File: extra/hardware/z280-s100/z280-s100.kicad_pcb (KiCad board)
At the start: 2 copper layers, 293.6 x 169.1 mm, 33 parts, among them J1 S-100 edge, J2 JTAG (1x6), J3 JP VPP, J4 JP A15, J5 JP A16, J6 JP A17/VDD, J7 JP PGM, J8 JP VDD, U1 Z280 (PLCC-68), U10 SRAM bank0 odd, U11 27SF020 even, U12 27SF020 odd, U13 MAX232, U14 DS1813 reset, U15 7805, U16 74HCT245 addr0, U17 74HCT245 addr1, U18 74HCT245 addr2, U19 74HCT245 status, U2 ATF1508 control, U20 74HCT245 control, U21 74HCT245 pHLDA, U22 SRAM bank1 even, U23 SRAM bank1 odd, U24 ATF1508 data, U3 74HC573 lo, U4 74HC573 hi, U9 SRAM bank0 even, Y1 24 MHz crystal

Commit message: PCB: through-hole PLCC sockets, rotated DIP-32 layout, fixed edge cuts
- PLCCs now mount in through-hole 0.1" sockets (68/84 pins, 4-sided) so
  there are real pads to route to
- DIP-32 SRAM/flash sockets rotated 90 and stacked per bank with vertical
  daylight instead of overlapping
- board outline gr_lines fixed to modern (stroke ...) syntax with correct
  layer numbers, and the project file migrated to the JSON format
Parts:
- U1: footprint PLCC-68 -> PLCC-68-SKT
- U2, U24: footprint PLCC-84 -> PLCC-84-SKT
- moved U14 261.9 mm to (270.0, 110.0)
- moved U15 261.9 mm to (270.0, 130.0)
- moved Y1 250.4 mm to (270.0, 90.0)
- moved U9 146.9 mm to (60.0, 40.0), turned to 90 degrees
- moved U10 142.7 mm to (60.0, 15.0), turned to 90 degrees
- moved U16 105.8 mm to (90.0, 130.0)
- moved U17 105.8 mm to (110.0, 130.0)
- moved U18 105.8 mm to (130.0, 130.0)
- moved U19 105.8 mm to (150.0, 130.0)
- moved U20 105.8 mm to (170.0, 130.0)
- moved U21 105.8 mm to (190.0, 130.0)
- moved U22 104.7 mm to (140.0, 40.0), turned to 90 degrees
- moved U23 98.7 mm to (140.0, 15.0), turned to 90 degrees
- moved U24 97.7 mm to (225.0, 85.0)
- moved U11 76.2 mm to (225.0, 40.0), turned to 90 degrees
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